File: pcb_layout/valve_driver.sch (KiCad schematic (older format))
At the start: 10 parts, among them J6 Conn_01x02, J7 Conn_01x02, Q1 Q_PMOS_GSD, Q2 Q_PMOS_GSD, U2 HCPL2731

Commit message: new pcb
Parts:
- R1, R2, R4: value 2.3k -> 2.32k
- R3: value 23.k -> 2.32k
Changed lines of the file:
@@
 AR Path="/5B406E77/5B4046E0" Ref="U4"  Part="1"
 AR Path="/5B406E7B/5B4046E0" Ref="U5"  Part="1"
-F 0 "U2" H 3600 4000 50  0000 L CNN
+F 0 "U5" H 3600 4000 50  0000 L CNN
 F 1 "HCPL2731" H 3600 3880 50  0000 L CNN
 F 2 "Housings_DIP:DIP-8_W7.62mm_Socket" H 3475 3950 50  0001 C CNN
@@
 AR Path="/5B406E77/5B4047D2" Ref="R9"  Part="1"
 AR Path="/5B406E7B/5B4047D2" Ref="R13"  Part="1"
-F 0 "R1" V 3430 1850 50  0000 C CNN
-F 1 "2.3k" V 3350 1850 50  0000 C CNN
+F 0 "R13" V 3430 1850 50  0000 C CNN
+F 1 "2.32k" V 3350 1850 50  0000 C CNN
 F 2 "Resistors_SMD:R_0805_HandSoldering" V 3280 1850 50  0001 C CNN
 F 3 "" H 3350 1850 50  0001 C CNN
@@
 AR Path="/5B406E77/5B404810" Ref="#PWR020"  Part="1"
 AR Path="/5B406E7B/5B404810" Ref="#PWR027"  Part="1"
-F 0 "#PWR06" H 3350 2450 50  0001 C CNN
+F 0 "#PWR027" H 3350 2450 50  0001 C CNN
 F 1 "GND" H 3350 2550 50  0000 C CNN
 F 2 "" H 3350 2700 50  0001 C CNN
@@
 AR Path="/5B406E77/5B404828" Ref="#PWR021"  Part="1"
 AR Path="/5B406E7B/5B404828" Ref="#PWR028"  Part="1"
-F 0 "#PWR07" H 3550 2450 50  0001 C CNN
+F 0 "#PWR028" H 3550 2450 50  0001 C CNN
 F 1 "GND" H 3550 2550 50  0000 C CNN
 F 2 "" H 3550 2700 50  0001 C CNN
@@
 AR Path="/5B406E77/5B4049D3" Ref="R11"  Part="1"
 AR Path="/5B406E7B/5B4049D3" Ref="R15"  Part="1"
-F 0 "R3" V 3630 1850 50  0000 C CNN
-F 1 "23.k" V 3550 1850 50  0000 C CNN
+F 0 "R15" V 3630 1850 50  0000 C CNN
+F 1 "2.32k" V 3550 1850 50  0000 C CNN
 F 2 "Resistors_SMD:R_0805_HandSoldering" V 3480 1850 50  0001 C CNN
 F 3 "" H 3550 1850 50  0001 C CNN
@@
 AR Path="/5B406E77/5B404DC3" Ref="#PWR022"  Part="1"
 AR Path="/5B406E7B/5B404DC3" Ref="#PWR029"  Part="1"
-F 0 "#PWR08" H 4050 2450 50  0001 C CNN
+F 0 "#PWR029" H 4050 2450 50  0001 C CNN
 F 1 "GND" H 4050 2550 50  0000 C CNN
 F 2 "" H 4050 2700 50  0001 C CNN
@@
 AR Path="/5B406E77/5B405242" Ref="R10"  Part="1"
 AR Path="/5B406E7B/5B405242" Ref="R14"  Part="1"
-F 0 "R2" V 3430 3500 50  0000 C CNN
-F 1 "2.3k" V 3350 3500 50  0000 C CNN
+F 0 "R14" V 3430 3500 50  0000 C CNN
+F 1 "2.32k" V 3350 3500 50  0000 C CNN
 F 2 "Resistors_SMD:R_0805_HandSoldering" V 3280 3500 50  0001 C CNN
 F 3 "" H 3350 3500 50  0001 C CNN
@@
 AR Path="/5B406E77/5B405248" Ref="#PWR023"  Part="1"
 AR Path="/5B406E7B/5B405248" Ref="#PWR030"  Part="1"
-F 0 "#PWR09" H 3350 4100 50  0001 C CNN
+F 0 "#PWR030" H 3350 4100 50  0001 C CNN
 F 1 "GND" H 3350 4200 50  0000 C CNN
 F 2 "" H 3350 4350 50  0001 C CNN
@@
 AR Path="/5B406E77/5B40524E" Ref="#PWR024"  Part="1"
 AR Path="/5B406E7B/5B40524E" Ref="#PWR031"  Part="1"
-F 0 "#PWR010" H 3550 4100 50  0001 C CNN
+F 0 "#PWR031" H 3550 4100 50  0001 C CNN
 F 1 "GND" H 3550 4200 50  0000 C CNN
 F 2 "" H 3550 4350 50  0001 C CNN
@@
 AR Path="/5B406E77/5B405255" Ref="R12"  Part="1"
 AR Path="/5B406E7B/5B405255" Ref="R16"  Part="1"
-F 0 "R4" V 3630 3500 50  0000 C CNN
-F 1 "2.3k" V 3550 3500 50  0000 C CNN
+F 0 "R16" V 3630 3500 50  0000 C CNN
+F 1 "2.32k" V 3550 3500 50  0000 C CNN
 F 2 "Resistors_SMD:R_0805_HandSoldering" V 3480 3500 50  0001 C CNN
 F 3 "" H 3550 3500 50  0001 C CNN
@@
 AR Path="/5B406E77/5B405267" Ref="#PWR025"  Part="1"
 AR Path="/5B406E7B/5B405267" Ref="#PWR032"  Part="1"
-F 0 "#PWR011" H 4050 4100 50  0001 C CNN
+F 0 "#PWR032" H 4050 4100 50  0001 C CNN
 F 1 "GND" H 4050 4200 50  0000 C CNN
 F 2 "" H 4050 4350 50  0001 C CNN
@@
 AR Path="/5B406E77/5B405304" Ref="U4"  Part="2"
 AR Path="/5B406E7B/5B405304" Ref="U5"  Part="2"
-F 0 "U2" H 3600 2350 50  0000 L CNN
+F 0 "U5" H 3600 2350 50  0000 L CNN
 F 1 "HCPL2731" H 3600 2230 50  0000 L CNN
 F 2 "Housings_DIP:DIP-8_W7.62mm_Socket" H 3475 2300 50  0001 C CNN
@@
 AR Path="/5B406E77/5B45A157" Ref="Q5"  Part="1"
 AR Path="/5B406E7B/5B45A157" Ref="Q7"  Part="1"
-F 0 "Q1" H 4150 2050 50  0000 L CNN
+F 0 "Q7" H 4150 2050 50  0000 L CNN
 F 1 "Q_PMOS_GSD" H 4150 1950 50  0000 L CNN
 F 2 "TO_SOT_Packages_SMD:SOT-23W_Handsoldering" H 4150 2100 50  0001 C CNN
@@
 AR Path="/5B406E77/5B45A1AF" Ref="Q6"  Part="1"
 AR Path="/5B406E7B/5B45A1AF" Ref="Q8"  Part="1"
-F 0 "Q2" H 4150 3700 50  0000 L CNN
+F 0 "Q8" H 4150 3700 50  0000 L CNN
 F 1 "Q_PMOS_GSD" H 4150 3600 50  0000 L CNN
 F 2 "TO_SOT_Packages_SMD:SOT-23W_Handsoldering" H 4150 3750 50  0001 C CNN
@@
 AR Path="/5B406E77/5B45A4D8" Ref="D3"  Part="1"
 AR Path="/5B406E7B/5B45A4D8" Ref="D4"  Part="1"
-F 0 "D1" H 5950 2800 50  0000 C CNN
+F 0 "D4" H 5950 2800 50  0000 C CNN
 F 1 "D_Schottky_x2_ACom_KKA" H 5900 3000 50  0000 C CNN
 F 2 "TO_SOT_Packages_SMD:SOT-23_Handsoldering" H 5900 2900 50  0001 C CNN
@@
 AR Path="/5B406E77/5B45A5E4" Ref="#PWR026"  Part="1"
 AR Path="/5B406E7B/5B45A5E4" Ref="#PWR033"  Part="1"
-F 0 "#PWR012" H 6100 2850 50  0001 C CNN
+F 0 "#PWR033" H 6100 2850 50  0001 C CNN
 F 1 "GND" H 6100 2950 50  0000 C CNN
 F 2 "" H 6100 3100 50  0001 C CNN
@@
 AR Path="/5B406E77/5B48319E" Ref="J10"  Part="1"
 AR Path="/5B406E7B/5B48319E" Ref="J12"  Part="1"
-F 0 "J6" H 4250 2500 50  0000 C CNN
+F 0 "J12" H 4250 2500 50  0000 C CNN
 F 1 "Conn_01x02" H 4250 2200 50  0000 C CNN
 F 2 "Pin_Headers:Pin_Header_Straight_1x02_Pitch2.00mm" H 4250 2400 50  0001 C CNN
@@
 AR Path="/5B406E77/5B4831E4" Ref="J11"  Part="1"
 AR Path="/5B406E7B/5B4831E4" Ref="J13"  Part="1"
-F 0 "J7" H 4250 4150 50  0000 C CNN
+F 0 "J13" H 4250 4150 50  0000 C CNN
 F 1 "Conn_01x02" H 4250 3850 50  0000 C CNN
 F 2 "Pin_Headers:Pin_Header_Straight_1x02_Pitch2.00mm" H 4250 4050 50  0001 C CNN
