File: pcb_layout/valve_testing.sch (KiCad schematic (older format))
At the start: 8 parts, among them J1 Conn_01x02, J2 Conn_01x03, J3 Conn_01x03, J4 Conn_01x02, J5 Conn_01x02, U1 74HC595

Commit message: new pcb
Parts:
- removed J1: Conn_01x02, Wire_Connections_Bridges:WireConnection_2.00mmDrill, symbol Conn_01x02
- removed J2, J3: Conn_01x03, Pin_Headers:Pin_Header_Straight_1x03_Pitch2.54mm, symbol Conn_01x03
- added J1: Barrel_Jack, Connectors:BARREL_JACK, symbol Barrel_Jack
- added J2, J3: Conn_01x04, Pin_Headers:Pin_Header_Angled_1x04_Pitch2.54mm, symbol Conn_01x04
Connections:
- wire segments 42 -> 41
Changed lines of the file:
@@
 	1    0    0    -1
 $EndComp
-Text GLabel 2950 4700 0    60   Input ~ 0
+Text GLabel 3150 4600 2    60   Input ~ 0
 Vcc_12V
 $Comp
@@
 	1    0    0    -1
 $EndComp
-Wire Wire Line
-	7550 1750 7800 1750
-Wire Wire Line
-	7550 1850 7800 1850
-Wire Wire Line
-	7550 1950 7800 1950
-Wire Wire Line
-	7550 2050 7800 2050
-Wire Wire Line
-	7550 2150 7800 2150
-Wire Wire Line
-	7550 2250 7800 2250
-Wire Wire Line
-	7550 2350 7800 2350
-Wire Wire Line
-	7550 2450 7800 2450
-Wire Wire Line
-	8450 1600 8200 1600
-Wire Wire Line
-	8450 1850 8200 1850
-Wire Wire Line
-	8450 2600 8200 2600
-Wire Wire Line
-	8450 2850 8200 2850
-Wire Wire Line
-	9650 2850 9400 2850
-Wire Wire Line
-	9650 2600 9400 2600
-Wire Wire Line
-	9650 1850 9400 1850
-Wire Wire Line
-	9650 1600 9400 1600
-Wire Wire Line
-	4600 2100 5100 2100
-Wire Wire Line
-	6150 1750 5700 1750
-Wire Wire Line
-	6150 1950 5700 1950
-Wire Wire Line
-	6150 2250 5700 2250
-Wire Wire Line
-	2000 3500 1400 3500
-Wire Wire Line
-	2000 3100 1700 3100
-Wire Wire Line
-	6150 2550 6150 2350
-Wire Wire Line
-	6150 2050 5700 2050
-Wire Wire Line
-	6550 1650 6550 1400
-Wire Wire Line
-	4600 2500 5100 2500
-Wire Wire Line
-	6850 4750 6500 4750
-Wire Wire Line
-	6850 4850 6500 4850
-Wire Wire Line
-	1400 3900 1400 3800
 Text Label 5700 2050 0    60   ~ 0
 SRCLR
-Wire Wire Line
-	4600 2200 5100 2200
 Text Label 5100 2500 2    60   ~ 0
 dataPin
-Wire Wire Line
-	4600 2300 5100 2300
 Text Label 5100 2100 2    60   ~ 0
 SRCLR
@@
 	1    0    0    -1
 $EndComp
-Wire Wire Line
-	2000 3100 2000 3300
-Connection ~ 2000 3200
-Wire Wire Line
-	7700 2650 7550 2650
-Wire Wire Line
-	7700 2750 7700 3200
-Wire Wire Line
-	7700 3200 5100 3200
-Wire Wire Line
-	5100 3200 5100 2500
-$Comp
-L Conn_01x02 J1
-U 1 1 5B459E71
-P 3400 4700
-F 0 "J1" H 3400 4800 50  0000 C CNN
-F 1 "Conn_01x02" H 3400 4500 50  0000 C CNN
-F 2 "Wire_Connections_Bridges:WireConnection_2.00mmDrill" H 3400 4700 50  0001 C CNN
-F 3 "" H 3400 4700 50  0001 C CNN
-	1    3400 4700
-	1    0    0    -1
-$EndComp
-Wire Wire Line
-	2950 4700 3200 4700
-Wire Wire Line
-	3200 4800 2950 4800
 $Comp
 L Conn_01x02 J5
@@
 $EndComp
 $Comp
-L Conn_01x03 J2
-U 1 1 5B48D3ED
-P 4400 4300
-F 0 "J2" H 4400 4500 50  0000 C CNN
-F 1 "Conn_01x03" H 4400 4100 50  0000 C CNN
-F 2 "Pin_Headers:Pin_Header_Straight_1x03_Pitch2.54mm" H 4400 4300 50  0001 C CNN
-F 3 "" H 4400 4300 50  0001 C CNN
-	1    4400 4300
+L Conn_01x04 J2
+U 1 1 5B6CCCC7
+P 4300 4300
+F 0 "J2" H 4300 4500 50  0000 C CNN
+F 1 "Conn_01x04" H 4300 4000 50  0000 C CNN
+F 2 "Pin_Headers:Pin_Header_Angled_1x04_Pitch2.54mm" H 4300 4300 50  0001 C CNN
+F 3 "" H 4300 4300 50  0001 C CNN
+	1    4300 4300
 	0    -1   -1   0
 $EndComp
-$Comp
-L Conn_01x03 J3
-U 1 1 5B48D489
-P 4400 5200
-F 0 "J3" H 4400 5400 50  0000 C CNN
-F 1 "Conn_01x03" H 4400 5000 50  0000 C CNN
-F 2 "Pin_Headers:Pin_Header_Straight_1x03_Pitch2.54mm" H 4400 5200 50  0001 C CNN
-F 3 "" H 4400 5200 50  0001 C CNN
-	1    4400 5200
-	0    1    1    0
-$EndComp
+Wire Wire Line
+	7550 1750 7800 1750
+Wire Wire Line
+	7550 1850 7800 1850
+Wire Wire Line
+	7550 1950 7800 1950
+Wire Wire Line
+	7550 2050 7800 2050
+Wire Wire Line
+	7550 2150 7800 2150
+Wire Wire Line
+	7550 2250 7800 2250
+Wire Wire Line
+	7550 2350 7800 2350
+Wire Wire Line
+	7550 2450 7800 2450
+Wire Wire Line
+	8450 1600 8200 1600
+Wire Wire Line
+	8450 1850 8200 1850
+Wire Wire Line
+	8450 2600 8200 2600
+Wire Wire Line
+	8450 2850 8200 2850
+Wire Wire Line
+	9650 2850 9400 2850
+Wire Wire Line
+	9650 2600 9400 2600
+Wire Wire Line
+	9650 1850 9400 1850
+Wire Wire Line
+	9650 1600 9400 1600
+Wire Wire Line
+	4600 2100 5100 2100
+Wire Wire Line
+	6150 1750 5700 1750
+Wire Wire Line
+	6150 1950 5700 1950
+Wire Wire Line
+	6150 2250 5700 2250
+Wire Wire Line
+	2000 3500 1400 3500
+Wire Wire Line
+	2000 3100 1700 3100
+Wire Wire Line
+	6150 2550 6150 2350
+Wire Wire Line
+	6150 2050 5700 2050
+Wire Wire Line
+	6550 1650 6550 1400
+Wire Wire Line
+	4600 2500 5100 2500
+Wire Wire Line
+	6850 4750 6500 4750
+Wire Wire Line
+	6850 4850 6500 4850
+Wire Wire Line
+	1400 3900 1400 3800
+Wire Wire Line
+	4600 2200 5100 2200
+Wire Wire Line
+	4600 2300 5100 2300
+Wire Wire Line
+	2000 3100 2000 3300
+Connection ~ 2000 3200
+Wire Wire Line
+	7700 2650 7550 2650
+Wire Wire Line
+	7700 2750 7700 3200
+Wire Wire Line
+	7700 3200 5100 3200
+Wire Wire Line
+	5100 3200 5100 2500
+Wire Wire Line
+	2950 4700 2950 5050
 Wire Wire Line
 	2950 4500 4500 4500
+Connection ~ 4200 4500
+Connection ~ 4300 4500
 Connection ~ 4400 4500
-Wire Wire Line
-	2950 4500 2950 4700
-Connection ~ 4300 4500
+$Comp
+L Conn_01x04 J3
+U 1 1 5B6CD2BC
+P 4300 5200
+F 0 "J3" H 4300 5400 50  0000 C CNN
+F 1 "Conn_01x04" H 4300 4900 50  0000 C CNN
+F 2 "Pin_Headers:Pin_Header_Angled_1x04_Pitch2.54mm" H 4300 5200 50  0001 C CNN
+F 3 "" H 4300 5200 50  0001 C CNN
+	1    4300 5200
+	0    -1   1    0
+$EndComp
 Wire Wire Line
 	2950 5000 4500 5000
 Connection ~ 4400 5000
-Wire Wire Line
-	2950 4800 2950 5050
 Connection ~ 4300 5000
 Connection ~ 2950 5000
+Connection ~ 4200 5000
+$Comp
+L Barrel_Jack J1
+U 1 1 5B6CD8B7
+P 2650 4700
+F 0 "J1" H 2650 4910 50  0000 C CNN
+F 1 "Barrel_Jack" H 2650 4525 50  0000 C CNN
+F 2 "Connectors:BARREL_JACK" H 2700 4660 50  0001 C CNN
+F 3 "" H 2700 4660 50  0001 C CNN
+	1    2650 4700
+	1    0    0    -1
+$EndComp
+Wire Wire Line
+	2950 4500 2950 4600
+Wire Wire Line
+	2950 4600 3150 4600
+Connection ~ 2950 4800
 $EndSCHEMATC
