File: pcb_layout/valve_testing.kicad_pcb (KiCad board)
At the start: 2 copper layers, 73.7 x 55.9 mm, 49 parts, among them J1 Conn_01x02, J10 Conn_01x02, J11 Conn_01x02, J12 Conn_01x02, J13 Conn_01x02, J2 Conn_01x03, J3 Conn_01x03, J4 Conn_01x02, J5 Conn_01x02, J6 Conn_01x02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

Commit message: new pcb
Parts:
- J1: value Conn_01x02 -> Barrel_Jack; footprint Wire_Connections_Bridges:WireConnection_2.00mmDrill -> Connectors:BARREL_JACK
- J2, J3: value Conn_01x03 -> Conn_01x04
- R1, R10, R12, R13, R14, R16, R2, R4, R5, R6, R8, R9: value 2.3k -> 2.32k
- R11, R15, R3, R7: value 23.k -> 2.32k
- moved J4 20.8 mm to (150.5, 83.1)
- moved C1 20.7 mm to (151.8, 85.6)
- moved J1 11.8 mm to (86.4, 76.8), turned to 0 degrees
- moved J2 9.56 mm to (91.4, 64.1)
- moved J3 8.79 mm to (88.9, 64.1)
- moved J5 7.67 mm to (147.3, 58.3)
Routing:
- net GND: track 39.5 -> 52.4 mm
- net Net-(J5-Pad1): track 8.25 -> 16.6 mm
- net /dataPin: track 24.8 -> 33.1 mm
- net VCC: track 100.0 -> 94.6 mm, vias 1 -> 0
- net Vcc_12V: track 185.3 -> 190.4 mm

Commit message: Add more details on how to solder and assemble
Parts:
- moved J3 12.1 mm to (90.2, 52.1), turned to 90 degrees
- moved J2 9.61 mm to (90.2, 54.6), turned to 90 degrees
Routing:
- net Vcc_12V: track 190.4 -> 228.3 mm
- net GND: track 52.4 -> 15.3 mm
Other:
- board text added: "5V"
- board text added: "GND"
Changed lines of the file:
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@@
   (general
     (links 115)
-    (no_connects 3)
-    (area 78.530379 47.48 158.750001 104.648001)
+    (no_connects 4)
+    (area 78.530379 47.26838 158.750001 104.648001)
     (thickness 1.6)
-    (drawings 14)
-    (tracks 238)
+    (drawings 18)
+    (tracks 234)
     (zones 0)
     (modules 49)
@@
   (page A4)
   (layers
-    (0 F.Cu signal)
+    (0 F.Cu signal hide)
     (31 B.Cu signal)
     (32 B.Adhes user hide)
@@
   )
   (setup
-    (last_trace_width 0.508)
+    (last_trace_width 0.3048)
     (user_trace_width 0.2032)
     (user_trace_width 0.254)
@@
   )
   (module Pin_Headers:Pin_Header_Straight_1x03_Pitch2.54mm (layer F.Cu)
-    (at 91.44 64.135)
+    (at 90.17 54.61 90)
     (descr "Through hole straight pin header, 1x03, 2.54mm pitch, single row")
     (tags "Through hole pin header THT 1x03 2.54mm single row")
-    (fp_text reference J2 (at 0 -2.33) (layer F.SilkS)
-      (effects (font (size 1 1) (thickness 0.15)))
-    )
-    (fp_text value Conn_01x04 (at 0 7.41) (layer F.Fab)
+    (fp_text reference J2 (at 0 -2.33 90) (layer F.SilkS)
+      (effects (font (size 1 1) (thickness 0.15)))
+    )
+    (fp_text value Conn_01x04 (at 0 7.41 90) (layer F.Fab)
       (effects (font (size 1 1) (thickness 0.15)))
     )
@@
     (fp_line (start 1.8 6.85) (end 1.8 -1.8) (layer F.CrtYd) (width 0.05))
     (fp_line (start 1.8 -1.8) (end -1.8 -1.8) (layer F.CrtYd) (width 0.05))
-    (fp_text user %R (at 0 2.54 90) (layer F.Fab)
-      (effects (font (size 1 1) (thickness 0.15)))
-    )
-    (pad 1 thru_hole rect (at 0 0) (size 1.7 1.7) (drill 1) (layers *.Cu *.Mask)
-      (net 2 Vcc_12V))
-    (pad 2 thru_hole oval (at 0 2.54) (size 1.7 1.7) (drill 1) (layers *.Cu *.Mask)
-      (net 2 Vcc_12V))
-    (pad 3 thru_hole oval (at 0 5.08) (size 1.7 1.7) (drill 1) (layers *.Cu *.Mask)
+    (fp_text user %R (at 0 2.54 180) (layer F.Fab)
+      (effects (font (size 1 1) (thickness 0.15)))
+    )
+    (pad 1 thru_hole rect (at 0 0 90) (size 1.7 1.7) (drill 1) (layers *.Cu *.Mask)
+      (net 2 Vcc_12V))
+    (pad 2 thru_hole oval (at 0 2.54 90) (size 1.7 1.7) (drill 1) (layers *.Cu *.Mask)
+      (net 2 Vcc_12V))
+    (pad 3 thru_hole oval (at 0 5.08 90) (size 1.7 1.7) (drill 1) (layers *.Cu *.Mask)
       (net 2 Vcc_12V))
     (model ${KISYS3DMOD}/Pin_Headers.3dshapes/Pin_Header_Straight_1x03_Pitch2.54mm.wrl
@@
   )
   (module Pin_Headers:Pin_Header_Straight_1x03_Pitch2.54mm (layer F.Cu)
-    (at 88.9 64.135)
+    (at 90.17 52.07 90)
     (descr "Through hole straight pin header, 1x03, 2.54mm pitch, single row")
     (tags "Through hole pin header THT 1x03 2.54mm single row")
-    (fp_text reference J3 (at 0 -2.33) (layer F.SilkS)
-      (effects (font (size 1 1) (thickness 0.15)))
-    )
-    (fp_text value Conn_01x04 (at 0 7.41) (layer F.Fab)
+    (fp_text reference J3 (at 0 -2.33 90) (layer F.SilkS)
+      (effects (font (size 1 1) (thickness 0.15)))
+    )
+    (fp_text value Conn_01x04 (at 0 7.41 90) (layer F.Fab)
       (effects (font (size 1 1) (thickness 0.15)))
     )
@@
     (fp_line (start 1.8 6.85) (end 1.8 -1.8) (layer F.CrtYd) (width 0.05))
     (fp_line (start 1.8 -1.8) (end -1.8 -1.8) (layer F.CrtYd) (width 0.05))
-    (fp_text user %R (at 0 2.54 90) (layer F.Fab)
-      (effects (font (size 1 1) (thickness 0.15)))
-    )
-    (pad 1 thru_hole rect (at 0 0) (size 1.7 1.7) (drill 1) (layers *.Cu *.Mask)
-      (net 1 GND))
-    (pad 2 thru_hole oval (at 0 2.54) (size 1.7 1.7) (drill 1) (layers *.Cu *.Mask)
-      (net 1 GND))
-    (pad 3 thru_hole oval (at 0 5.08) (size 1.7 1.7) (drill 1) (layers *.Cu *.Mask)
+    (fp_text user %R (at 0 2.54 180) (layer F.Fab)
+      (effects (font (size 1 1) (thickness 0.15)))
+    )
+    (pad 1 thru_hole rect (at 0 0 90) (size 1.7 1.7) (drill 1) (layers *.Cu *.Mask)
+      (net 1 GND))
+    (pad 2 thru_hole oval (at 0 2.54 90) (size 1.7 1.7) (drill 1) (layers *.Cu *.Mask)
+      (net 1 GND))
+    (pad 3 thru_hole oval (at 0 5.08 90) (size 1.7 1.7) (drill 1) (layers *.Cu *.Mask)
       (net 1 GND))
     (model ${KISYS3DMOD}/Pin_Headers.3dshapes/Pin_Header_Straight_1x03_Pitch2.54mm.wrl
@@
     (pad 3 thru_hole rect (at 3.2004 4.699) (size 3.50012 3.50012) (drill oval 2.99974 1.00076) (layers *.Cu *.Mask)
       (net 1 GND))
+  )
+  (gr_text GND (at 128.524 102.616) (layer B.SilkS)
+    (effects (font (size 1 1) (thickness 0.1)) (justify mirror))
+  )
+  (gr_text 5V (at 125.984 102.616) (layer B.SilkS)
+    (effects (font (size 1 1) (thickness 0.1)) (justify mirror))
+  )
+  (gr_text GND (at 128.524 102.616) (layer F.SilkS)
+    (effects (font (size 1 1) (thickness 0.1)))
+  )
+  (gr_text 5V (at 125.857 102.616) (layer F.SilkS)
+    (effects (font (size 1 1) (thickness 0.1)))
   )
   (gr_line (start 157.48 51.435) (end 157.48 50.165) (angle 90) (layer Edge.Cuts) (width 0.15))
@@
   (gr_line (start 155.575 48.26) (end 85.725 48.26) (angle 90) (layer Edge.Cuts) (width 0.15))
   (gr_line (start 85.725 104.14) (end 155.575 104.14) (angle 90) (layer Edge.Cuts) (width 0.15))
-  (segment (start 88.265 63.5) (end 88.265 69.85) (width 2.54) (layer B.Cu) (net 1) (status 400000))
-  (segment (start 86.36 81.915) (end 86.36 71.755) (width 2.54) (layer B.Cu) (net 1))
-  (segment (start 86.36 71.755) (end 88.265 69.85) (width 2.54) (layer B.Cu) (net 1))
-  (segment (start 86.36 81.915) (end 93.345 81.915) (width 2.54) (layer B.Cu) (net 1))
-  (segment (start 88.265 63.5) (end 88.265 69.85) (width 2.54) (layer F.Cu) (net 1))
-  (segment (start 86.36 71.755) (end 88.265 69.85) (width 2.54) (layer F.Cu) (net 1))
-  (segment (start 86.36 81.915) (end 93.345 81.915) (width 2.54) (layer F.Cu) (net 1))
-  (segment (start 86.36 81.915) (end 86.36 71.755) (width 2.54) (layer F.Cu) (net 1))
-  (segment (start 101.52 82.423) (end 99.568 82.423) (width 0.508) (layer B.Cu) (net 2) (status 400000))
+  (segment (start 86.56066 76.835) (end 86.56066 78.53426) (width 2.54) (layer F.Cu) (net 1))
+  (segment (start 86.56066 78.53426) (end 89.5604 81.534) (width 2.54) (layer F.Cu) (net 1))
+  (segment (start 86.56066 78.53426) (end 89.5604 81.534) (width 2.54) (layer B.Cu) (net 1))
+  (segment (start 90.17 52.07) (end 95.25 52.07) (width 2.54) (layer B.Cu) (net 1))
+  (segment (start 92.56014 76.835) (end 93.98 76.835) (width 2.54) (layer F.Cu) (net 2))
+  (segment (start 93.98 76.835) (end 94.615 76.2) (width 2.54) (layer F.Cu) (net 2))
+  (segment (start 94.615 76.2) (end 94.615 55.245) (width 2.54) (layer F.Cu) (net 2))
+  (segment (start 92.56014 76.835) (end 92.56014 55.64886) (width 2.54) (layer F.Cu) (net 2))
+  (segment (start 92.41028 55.499) (end 90.17 55.499) (width 2.54) (layer F.Cu) (net 2))
+  (segment (start 92.56014 55.64886) (end 92.41028 55.499) (width 2.54) (layer F.Cu) (net 2))
+  (segment (start 93.98 76.835) (end 94.615 76.2) (width 2.54) (layer B.Cu) (net 2))
+  (segment (start 94.615 76.2) (end 94.615 55.245) (width 2.54) (layer B.Cu) (net 2))
+  (segment (start 92.56014 76.835) (end 92.56014 55.64886) (width 2.54) (layer B.Cu) (net 2))
+  (segment (start 92.41028 55.499) (end 90.17 55.499) (width 2.54) (layer B.Cu) (net 2))
+  (segment (start 92.56014 55.64886) (end 92.41028 55.499) (width 2.54) (layer B.Cu) (net 2))
+  (segment (start 101.52 82.423) (end 99.568 82.423) (width 0.508) (layer B.Cu) (net 2))
   (segment (start 98.425 81.28) (end 98.425 77.978) (width 0.508) (layer B.Cu) (net 2))
   (segment (start 99.568 82.423) (end 98.425 81.28) (width 0.508) (layer B.Cu) (net 2))
-  (segment (start 93.70314 77.978) (end 95.25 77.978) (width 0.508) (layer B.Cu) (net 2) (status 400000))
+  (segment (start 93.70314 77.978) (end 95.25 77.978) (width 0.508) (layer B.Cu) (net 2))
   (segment (start 95.25 77.978) (end 98.425 77.978) (width 0.508) (layer B.Cu) (net 2))
   (segment (start 98.425 77.978) (end 108.585 77.978) (width 0.508) (layer B.Cu) (net 2))
-  (segment (start 93.70314 77.978) (end 92.56014 76.835) (width 0.508) (layer B.Cu) (net 2) (status C00000))
-  (segment (start 94.996 67.056) (end 92.56014 64.62014) (width 2.54) (layer B.Cu) (net 2))
-  (segment (start 94.996 75.692) (end 94.996 67.056) (width 2.54) (layer B.Cu) (net 2))
-  (segment (start 93.853 76.835) (end 94.996 75.692) (width 2.54) (layer B.Cu) (net 2))
-  (segment (start 92.56014 76.835) (end 93.853 76.835) (width 2.54) (layer B.Cu) (net 2))
-  (segment (start 92.56014 76.835) (end 92.56014 64.62014) (width 2.54) (layer B.Cu) (net 2))
-  (segment (start 92.56014 64.62014) (end 92.075 64.135) (width 2.54) (layer B.Cu) (net 2))
-  (segment (start 93.853 76.835) (end 94.996 75.692) (width 2.54) (layer F.Cu) (net 2))
-  (segment (start 94.996 67.056) (end 92.56014 64.62014) (width 2.54) (layer F.Cu) (net 2))
-  (segment (start 94.996 75.692) (end 94.996 67.056) (width 2.54) (layer F.Cu) (net 2))
-  (segment (start 92.56014 76.835) (end 92.56014 64.62014) (width 2.54) (layer F.Cu) (net 2))
-  (segment (start 92.56014 64.62014) (end 92.075 64.135) (width 2.54) (layer F.Cu) (net 2))
+  (segment (start 93.70314 77.978) (end 92.56014 76.835) (width 0.508) (layer B.Cu) (net 2))
   (segment (start 139.495 85.803) (end 138.11 85.803) (width 0.508) (layer B.Cu) (net 2))
   (segment (start 139.7 85.598) (end 139.495 85.803) (width 0.508) (layer B.Cu) (net 2))
